File: layout/mainboard/boat5.brd (EAGLE design)
At the start: 89 x 54 mm, 97 parts, among them IC3 ATMEGA2560-16AU, J1 AVR_SPI_PRG_6PTH, Q1 MOSFET-NCHANNELBSS138, Q2 MOSFET-PCHANNELSMD, Q3 MOSFET-PCHANNELSMD, Q4 MOSFET-PCHANNELSMD, Q5 MOSFET-NCHANNELBSS138, Q6 MOSFET-NCHANNELBSS138, Q7 MOSFET-NCHANNELBSS138, Q8 MOSFET-PCHANNELSMD, U1 MPU-9150, U2 VENUS638FLPX-L, U3 USD-SOCKETNEW, U4 HMC5883LSMD, Y1 CSTCE16M0V53-R0 16MHZ

Commit message: cleanup, porting to 2560
Routing:
- net GND: vias 79 -> 80
Changed lines of the file:
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@@
-<text x="87" y="37" size="1.016" layer="16" rot="MR90">ARDUSAILOR V5.1</text>
 <text x="87" y="37" size="1.016" layer="16" rot="MR90">ARDUSAILOR V5.1</text>
 <text x="87" y="37" size="1.016" layer="16" rot="MR90">ARDUSAILOR V5.1</text>
@@
 <via x="65" y="45" extent="1-16" drill="0.5"/>
 <via x="73" y="50" extent="1-16" drill="0.5"/>
-<via x="15" y="17" extent="1-16" drill="0.5"/>
-<via x="15" y="21" extent="1-16" drill="0.5"/>
-<via x="25" y="30" extent="1-16" drill="0.5"/>
-<via x="27.15" y="30" extent="1-16" drill="0.5"/>
+<via x="10" y="16" extent="1-16" drill="0.5"/>
+<via x="25" y="30" extent="1-16" drill="0.381"/>
+<via x="29.15" y="28" extent="1-16" drill="0.381"/>
 <contactref element="C9" pad="2"/>
 <via x="24.886" y="46.563" extent="1-16" drill="0.381"/>
@@
 <via x="79" y="8" extent="1-16" drill="0.381"/>
 <via x="81" y="8" extent="1-16" drill="0.381"/>
-<via x="19" y="21" extent="1-16" drill="0.5"/>
-<via x="19" y="17" extent="1-16" drill="0.5"/>
+<via x="17" y="24" extent="1-16" drill="0.5"/>
+<via x="29" y="22" extent="1-16" drill="0.5"/>
 <via x="50" y="20.9" extent="1-16" drill="0.381"/>
 <contactref element="U1" pad="9"/>
@@
 <via x="76" y="25" extent="1-16" drill="0.381"/>
 <via x="41.9" y="36.25" extent="1-16" drill="0.381"/>
+<via x="41" y="14" extent="1-16" drill="0.381"/>
+<via x="41" y="18" extent="1-16" drill="0.381"/>
 </signal>
 <signal name="SDA">
