File: layout/boat5.brd (EAGLE design)
At the start: 89 x 54 mm, 96 parts, among them IC3 ATMEGA2560-16AU, J1 AVR_SPI_PRG_6PTH, Q1 MOSFET-NCHANNELBSS138, Q2 MOSFET-PCHANNELSMD, Q3 MOSFET-PCHANNELSMD, Q4 MOSFET-PCHANNELSMD, Q5 MOSFET-NCHANNELBSS138, Q6 MOSFET-NCHANNELBSS138, Q7 MOSFET-NCHANNELBSS138, Q8 MOSFET-PCHANNELSMD, U1 MPU-9150, U2 VENUS638FLPX-L, U3 USD-SOCKETNEW, U4 HMC5883LSMD, Y1 CSTCE16M0V53-R0 16MHZ

Commit message: 5.1 final; submitted for build
Parts:
- removed D$3: SS1P3L, kolosy:MICROSMP
- removed D5: (no value), diode:SOD523
- added C31: 22uF, SparkFun-Capacitors:1206
- added C32: .1uF, SparkFun-Capacitors:0805
- added C33: DNP, SparkFun-Passives:0402-CAP
- C17: value 10uF -> 22uF
- C18: value .01uF -> DNP
- C19: value 1000pF -> .1uF; device SparkFun-Capacitors:0603-CAP -> SparkFun-Capacitors:0805
- L3: device kolosy:SLFXXXX -> kolosy:SLF7055
- R13: value 100k -> 10k
- R14: value 10k -> 56.8K
- R15: value 56.2k -> 10K
- U$2: value LM2374 -> TPS56X200
- moved C18 18.9 mm to (84.0, 22.0)
- moved C29 17.1 mm to (62.0, 20.0), turned to 270 degrees
- moved R13 16.0 mm to (78.0, 15.0), turned to 0 degrees
- moved R14 13.3 mm to (84.0, 20.0), turned to 180 degrees
- moved L3 12.7 mm to (83.2, 4.15), turned to 180 degrees
- moved R15 11.0 mm to (84.0, 18.0), turned to 0 degrees
- moved C20 9.17 mm to (76.0, 5.00), turned to 90 degrees
- moved C19 8.98 mm to (81.7, 15.3)
- moved U$2 7.81 mm to (84.0, 14.0)
- moved C17 7.58 mm to (84.0, 8.85), turned to 180 degrees
- moved R26 5.83 mm to (67.0, 39.0)
- moved JP1 3.00 mm to (86.0, 27.0)
- moved C24 1.41 mm to (40.0, 50.0), turned to 90 degrees
- turned JP2 to 90 degrees
Connections:
- removed net N$12: C18.1, D$3.C, L3.P$2, U$2.6
- new net N$19: C18.2, R14.1, R15.2, U$2.4
- new net N$32: C19.2, U$2.6
- net 3.3V: now also C33.1
- net 5V: now also C18.1, C31.1, L3.P$2, R14.2; no longer C19.1, D5.A, L3.P$1, R15.2
- net 5V_EN: no longer U$2.4
- net GND: now also C31.2, C32.2, R15.1, U$2.1; no longer D$3.A, R13.2, R14.1, U$2.2
- net N$11: now also C19.1, L3.P$1, U$2.2; no longer C18.2, D5.C, U$2.1
- net N$15: now also R13.2, U$2.5; no longer C19.2, R14.2, R15.1, U$2.3
- net N$17: now also C33.2
- net V_BATT: now also C32.1, U$2.3; no longer U$2.5
Routing:
- net 5V: track 126.6 -> 81.9 mm, vias 2 -> 0
- net RESET: track 124.4 -> 89.4 mm, vias 3 -> 5
- net WIND_EN: track 101.6 -> 67.8 mm, vias 8 -> 4
- net V_BATT: track 70.8 -> 47.5 mm
- net N$12: track 15.8 -> 0.00 mm
- net N$11: track 5.07 -> 16.4 mm, vias 0 -> 5
- net 5V_EN: track 56.4 -> 45.4 mm, vias 3 -> 2
- net N$19: track 0.00 -> 6.94 mm
- net TX_D0: track 27.8 -> 33.7 mm, vias 1 -> 2
- net BATT_SENS_EN: track 34.7 -> 29.4 mm
- net N$17: track 6.96 -> 10.3 mm
- net RUD_V: track 64.5 -> 61.9 mm
- net N$32: track 0.00 -> 2.07 mm
- net DTR: track 3.92 -> 2.00 mm
- net N$15: track 6.10 -> 7.83 mm
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
Commit message: more 3d stuff
Routing:
- net 3.3V: track 290.1 -> 293.1 mm
- net WINCH_EN: track 30.4 -> 29.2 mm
- net CS: track 74.6 -> 73.8 mm
- net GND: vias 79 -> 81
Changed lines of the file:
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@@
 <via x="65" y="45" extent="1-16" drill="0.5"/>
 <via x="73" y="50" extent="1-16" drill="0.5"/>
-<via x="15" y="17" extent="1-16" drill="0.5"/>
-<via x="15" y="21" extent="1-16" drill="0.5"/>
-<via x="25" y="30" extent="1-16" drill="0.5"/>
-<via x="27.15" y="30" extent="1-16" drill="0.5"/>
+<via x="15" y="17" extent="1-16" drill="0.381"/>
+<via x="15" y="21" extent="1-16" drill="0.381"/>
+<via x="25" y="30" extent="1-16" drill="0.381"/>
+<via x="27.15" y="30" extent="1-16" drill="0.381"/>
 <contactref element="C9" pad="2"/>
 <via x="24.886" y="46.563" extent="1-16" drill="0.381"/>
@@
 <via x="79" y="8" extent="1-16" drill="0.381"/>
 <via x="81" y="8" extent="1-16" drill="0.381"/>
-<via x="19" y="21" extent="1-16" drill="0.5"/>
-<via x="19" y="17" extent="1-16" drill="0.5"/>
+<via x="19" y="21" extent="1-16" drill="0.381"/>
+<via x="19" y="17" extent="1-16" drill="0.381"/>
 <via x="49" y="19.9" extent="1-16" drill="0.381"/>
 <contactref element="U1" pad="9"/>
@@
 <via x="76" y="25" extent="1-16" drill="0.381"/>
 <via x="41.9" y="36.25" extent="1-16" drill="0.381"/>
+<via x="63" y="12" extent="1-16" drill="0.5"/>
+<via x="63" y="6" extent="1-16" drill="0.5"/>
 </signal>
 <signal name="SDA">
@@
 <wire x1="34" y1="31.5" x2="35.35" y2="31.5" width="0.254" layer="1"/>
 <wire x1="35.35" y1="31.5" x2="35.85" y2="32" width="0.254" layer="1"/>
-<wire x1="35.85" y1="32" x2="38" y2="32" width="1.016" layer="1"/>
-<wire x1="38" y1="32" x2="42" y2="32" width="1.016" layer="1"/>
+<wire x1="35.85" y1="32" x2="40" y2="32" width="1.016" layer="1"/>
+<wire x1="40" y1="32" x2="42" y2="32" width="1.016" layer="1"/>
 <wire x1="42" y1="32" x2="43.5" y2="33.5" width="1.016" layer="1"/>
 <wire x1="43.5" y1="33.5" x2="45" y2="35" width="1.016" layer="1"/>
@@
 <wire x1="46" y1="38" x2="46" y2="36" width="0.254" layer="1"/>
 <wire x1="50" y1="29" x2="48" y2="29" width="0.254" layer="1"/>
-<wire x1="48" y1="29" x2="43.5" y2="33.5" width="0.254" layer="1"/>
+<wire x1="48" y1="29" x2="45" y2="32" width="0.254" layer="1"/>
+<wire x1="45" y1="32" x2="45" y2="34.5" width="0.254" layer="1"/>
+<wire x1="45" y1="34.5" x2="43.5" y2="33.5" width="0.254" layer="1"/>
 <wire x1="45" y1="35" x2="40" y2="35" width="0.254" layer="1"/>
 <wire x1="40" y1="35" x2="39" y2="36" width="0.254" layer="1"/>
@@
 <wire x1="32.45" y1="31.6" x2="32.45" y2="33.2" width="0.4064" layer="1"/>
 <wire x1="32.45" y1="33.2" x2="32.1" y2="33.55" width="0.4064" layer="1"/>
-<via x="26" y="35" extent="1-16" drill="0.6"/>
+<via x="26" y="35" extent="1-16" drill="0.381"/>
 <wire x1="26" y1="35" x2="29" y2="32" width="0.8128" layer="16"/>
 <wire x1="29" y1="32" x2="35.85" y2="32" width="0.8128" layer="16"/>
@@
 <wire x1="36.8" y1="24.75" x2="37" y2="25" width="0.6096" layer="1"/>
 <wire x1="37" y1="25" x2="37" y2="29" width="0.6096" layer="1"/>
-<wire x1="37" y1="29" x2="38" y2="30" width="0.6096" layer="1"/>
-<wire x1="38" y1="30" x2="38" y2="32" width="0.6096" layer="1"/>
+<wire x1="37" y1="29" x2="40" y2="32" width="0.6096" layer="1"/>
 <via x="22" y="39" extent="1-16" drill="0.5"/>
 <wire x1="22" y1="39" x2="26" y2="35" width="0.6096" layer="16"/>
@@
 <via x="33" y="42" extent="1-16" drill="0.381"/>
 <wire x1="33" y1="42" x2="38" y2="42" width="0.254" layer="16"/>
-<wire x1="38" y1="42" x2="40" y2="40" width="0.254" layer="16"/>
-<wire x1="40" y1="40" x2="45" y2="40" width="0.254" layer="16"/>
-<wire x1="45" y1="40" x2="46" y2="41" width="0.254" layer="16"/>
-<wire x1="46" y1="41" x2="49" y2="41" width="0.254" layer="16"/>
+<wire x1="38" y1="42" x2="39" y2="41" width="0.254" layer="16"/>
+<wire x1="39" y1="41" x2="49" y2="41" width="0.254" layer="16"/>
 <via x="49" y="41" extent="1-16" drill="0.381"/>
 <wire x1="49" y1="41" x2="47.5" y2="39.5" width="0.254" layer="1"/>
@@
 <wire x1="51" y1="35" x2="52" y2="34" width="0.254" layer="1"/>
 <via x="52" y="34" extent="1-16" drill="0.381"/>
-<via x="56" y="33" extent="1-16" drill="0.381"/>
-<wire x1="56" y1="33" x2="56" y2="42" width="0.254" layer="1"/>
-<via x="56" y="42" extent="1-16" drill="0.381"/>
-<wire x1="56" y1="42" x2="55" y2="42" width="0.254" layer="16"/>
-<wire x1="55" y1="42" x2="54" y2="43" width="0.254" layer="16"/>
+<via x="56" y="34" extent="1-16" drill="0.381"/>
+<wire x1="56" y1="34" x2="56" y2="41" width="0.254" layer="1"/>
+<via x="56" y="41" extent="1-16" drill="0.381"/>
+<wire x1="56" y1="41" x2="54" y2="43" width="0.254" layer="16"/>
 <wire x1="54" y1="43" x2="54" y2="44" width="0.254" layer="16"/>
 <wire x1="59.33" y1="48.04" x2="59.96" y2="48.04" width="0.254" layer="1"/>
@@
 <wire x1="55" y1="45" x2="54" y2="44" width="0.254" layer="16"/>
 <wire x1="52" y1="34" x2="53" y2="33" width="0.254" layer="16"/>
-<wire x1="53" y1="33" x2="56" y2="33" width="0.254" layer="16"/>
+<wire x1="53" y1="33" x2="55" y2="33" width="0.254" layer="16"/>
+<wire x1="55" y1="33" x2="56" y2="34" width="0.254" layer="16"/>
 </signal>
 <signal name="RUD_V">

Commit message: housing updates
Parts:
- turned R9 to 90 degrees
Routing:
- net 5V: track 81.9 -> 35.2 mm
- net 3.3V: track 293.1 -> 277.6 mm, vias 15 -> 17
- net WINCH_EN: track 29.2 -> 22.4 mm
- net SCL: track 57.7 -> 59.1 mm
- net RUD_EN: track 36.5 -> 35.3 mm
- net V_BATT_DIV: track 51.2 -> 52.0 mm
- net N$29: track 6.69 -> 7.28 mm
- net GND: vias 81 -> 92
Other:
- board text added: "ARDUSAILOR V5.2"
- board text removed: "ARDUSAILOR V5.1"
