File: layout/boat5.brd (EAGLE design)
At the start: 89 x 54 mm, 97 parts, among them IC3 ATMEGA2560-16AU, J1 AVR_SPI_PRG_6PTH, Q1 MOSFET-NCHANNELBSS138, Q2 MOSFET-PCHANNELSMD, Q3 MOSFET-PCHANNELSMD, Q4 MOSFET-PCHANNELSMD, Q5 MOSFET-NCHANNELBSS138, Q6 MOSFET-NCHANNELBSS138, Q7 MOSFET-NCHANNELBSS138, Q8 MOSFET-PCHANNELSMD, U1 MPU-9150, U2 VENUS638FLPX-L, U3 USD-SOCKETNEW, U4 HMC5883LSMD, Y1 CSTCE16M0V53-R0 16MHZ

Commit message: circuit updates, firmware tweaks
Parts:
- added C34: 470uF, SparkFun-Capacitors:CAP-PTH-5MM
- C13: value 250uF -> 4700uF
- C24: value 250uF -> 1000uF
Connections:
- net GND: now also C34.2
- net V_BATT: now also C34.1
Changed lines of the file:
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@@
 </element>
 <element name="R1" library="SparkFun-Resistors" package="0603-RES" value="100k" x="80" y="27" rot="R90"/>
-<element name="C13" library="SparkFun-Capacitors" package="CAP-PTH-5MM" value="250uF" x="76" y="49" rot="R270"/>
-<element name="C24" library="SparkFun-Capacitors" package="CAP-PTH-5MM" value="250uF" x="40" y="50" rot="R90"/>
+<element name="C13" library="SparkFun-Capacitors" package="CAP-PTH-5MM" value="4700uF" x="76" y="49" rot="R270"/>
+<element name="C24" library="SparkFun-Capacitors" package="CAP-PTH-5MM" value="1000uF" x="40" y="50" rot="R90"/>
 <element name="D$1" library="kolosy" package="MICROSMP" value="SS1P3L" x="51" y="47"/>
 <element name="D$2" library="kolosy" package="MICROSMP" value="SS1P3L" x="62" y="47"/>
@@
 <attribute name="VALUE" x="79.6705" y="34.107" size="0.4064" layer="27"/>
 </element>
+<element name="C34" library="SparkFun-Capacitors" package="CAP-PTH-5MM" value="470uF" x="79" y="21" rot="R270"/>
 </elements>
 <signals>
@@
 <via x="76.55" y="36.4" extent="1-16" drill="0.381"/>
 <via x="75.45" y="36.4" extent="1-16" drill="0.381"/>
+<contactref element="C34" pad="2"/>
 </signal>
 <signal name="SDA">
@@
 <contactref element="C17" pad="1"/>
 <contactref element="C32" pad="1"/>
+<contactref element="C34" pad="1"/>
 </signal>
 <signal name="N$8">

Commit message: new calibration params, other fixes
Parts:
- C10, C5, C7, C8: device SparkFun:0402-CAP -> SparkFun:0603-CAP
- C18, C33: value DNP -> 1nF
- L1: device SparkFun:C0402 -> SparkFun:0603
- R3, R4, R6: device SparkFun:0402-RES -> SparkFun:0603-RES
- moved C28 15.2 mm to (46.1, 40.4)
- moved R11 5.00 mm to (86.0, 48.0), turned to 0 degrees
- moved R5 4.50 mm to (86.0, 46.6), turned to 180 degrees
- moved R19 3.16 mm to (86.0, 45.0), turned to 180 degrees
- moved Q8 2.00 mm to (82.0, 46.0), turned to 0 degrees
- moved Q1 2.00 mm to (86.0, 40.0)
- moved Q7 2.00 mm to (82.0, 42.0)
- moved R24 2.00 mm to (86.0, 43.0)
- moved R27 2.00 mm to (82.0, 39.0)
- moved Y1 1.88 mm to (40.8, 17.7)
- moved R12 1.28 mm to (40.4, 20.1)
- moved C18 0.95 mm to (84.0, 21.1)
- moved D$2 0.65 mm to (62.6, 47.0)
- moved C34 0.63 mm to (78.4, 20.8)
- moved R14 0.50 mm to (84.0, 19.5)
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Routing:
- net V_BATT: track 47.5 -> 41.9 mm, vias 1 -> 0
- net V_BATT_DIV: track 52.0 -> 56.9 mm
- net N$29: track 7.28 -> 3.36 mm
- net XTAL2: track 6.71 -> 4.46 mm
- net N$30: track 5.11 -> 7.25 mm
- net VCC_EN: track 39.0 -> 41.0 mm
- net N$31: track 13.2 -> 15.2 mm
- net XTAL1: track 7.15 -> 5.33 mm
- net 3.3V: track 277.6 -> 275.8 mm
- net VBAT: track 18.9 -> 20.3 mm
- net N$19: track 6.94 -> 5.96 mm
- net N$23: track 16.9 -> 17.7 mm
- net N$9: track 7.99 -> 7.34 mm
- net GND: vias 92 -> 97

Commit message: pilot tuning
Parts:
- moved R8 4.24 mm to (67.5, 45.0), turned to 180 degrees
- moved C24 2.00 mm to (40.0, 48.0)
- moved C13 1.00 mm to (75.0, 49.0)
- moved R26 0.65 mm to (66.3, 39.0)
- moved R11 0.30 mm to (86.0, 48.3)
Routing:
- net PPS: track 15.8 -> 0.00 mm, vias 1 -> 0
- net RUD_EN: track 35.3 -> 29.2 mm
- net V_BATT_DIV: track 56.9 -> 54.6 mm
- net SCL: track 59.1 -> 57.2 mm
- net 3.3V: track 275.8 -> 277.2 mm, vias 17 -> 18
- net WS_1: track 50.1 -> 49.1 mm
- net CAM_EN: track 51.9 -> 51.0 mm
- net N$7: track 2.42 -> 3.27 mm
- net WN_V: track 85.5 -> 86.4 mm
- net WS_2: track 49.7 -> 48.9 mm
- net 5V: track 34.9 -> 34.2 mm
- net BATT_SENS_EN: track 29.4 -> 28.7 mm
- net N$31: track 15.2 -> 15.9 mm
- net WIND_EN: track 67.8 -> 68.4 mm
- net GND: vias 97 -> 104
Other:
- board text added: "ARDUSAILOR V5.3"
- board text removed: "ARDUSAILOR V5.2"
