File: layout/boat5.sch (EAGLE design)
At the start: 74 parts, among them IC3 ATMEGA2560-16AU, Q1 60V, Q2 60V, U1 MPU-9150, U2 VENUS638FLPX-L, U3 USD-SOCKETNEW, Y1 CSTCE16M0V53-R0 16MHZ

Commit message: first pass at routing
Parts:
- added C25: .1uF, SparkFun:CAP0402-CAP
- added C26: .22uF, SparkFun:CAP0402-CAP
- added C27: 4.7uF, SparkFun:CAP0402-CAP
- added R10, R2: DNP, SparkFun:RESISTOR0402-RES
- added U4: HMC5883LSMD, SparkFun:HMC5883LSMD
- C9: device SparkFun:CAP_POLPTH4 -> SparkFun:CAP_POLEN_J2
Connections:
- removed net PA4: IC3.(AD4)PA4
- removed net PA5: IC3.(AD5)PA5
- new net N$13: C26.2, U4.SETC
- new net N$16: C27.1, U4.C1
- new net N$3: C26.1, U4.SETP
- net GND: now also C25.2, C27.2, U4.GND@1, U4.GND@2
- net RUD_EN: now also IC3.(AD4)PA4
- net SCL: now also R2.1, U4.SCL
- net SDA: now also R10.1, U4.SDA
- net VCC: now also C25.1, R10.2, R2.2, U4.S1, U4.VDD, U4.VDDIO
- net WINCH_EN: now also IC3.(AD5)PA5

Commit message: boat v5
Parts:
- removed Q2: 60V, transistor-power:PMOSFET_NTO220BV
- removed RN5: 10K, resistor-dil:4R-NCAT16
- added C28: 10nF, SparkFun-Passives:CAP0402-CAP
- added J1: AVR_SPI_PRG_6PTH, SparkFun-Connectors:AVR_SPI_PRG_6PTH
- added Q3, Q4: MOSFET-PCHANNELSMD, SparkFun-DiscreteSemi:MOSFET-PCHANNELSMD
- added Q5, Q6: MOSFET-NCHANNELBSS138, SparkFun-DiscreteSemi:MOSFET-NCHANNELBSS138
- added R19: 10k, SparkFun-Resistors:RESISTOR0603
- added R20, R21: 100k, SparkFun-Resistors:RESISTOR0603
- added R22, R23, R24: 100R, SparkFun-Resistors:RESISTOR0603
- Q1: value 60V -> MOSFET-NCHANNELBSS138; device transistor-power:PMOSFET_NTO220BV -> SparkFun-DiscreteSemi:MOSFET-NCHANNELBSS138
Connections:
- removed net PC6: IC3.(A14)PC6
- removed net PC7: IC3.(A15)PC7
- removed net RX1: U2.RXD1
- removed net TX1: U2.TXD1
- removed net VCC: C12.1, C14.1, C15.1, C22.1, C23.+, C25.1, D4.C, IC3.AVCC, IC3.VCC, IC3.VCC1, IC3.VCC2, IC3.VCC3, R10.2, R16.2, R18.1, R2.2, RN1B.2, RN1C.2, RN5A.2, U$1.VOS, U$6.P$2, U4.S1, U4.VDD, U4.VDDIO
- new net CAM_EN: IC3.(A14)PC6, R23.2
- new net GPS_EN: IC3.(A15)PC7, R22.2
- new net GPS_PWR: C5.1, C6.+, C8.1, L1.1, Q3.D, R3.2, SJ2.1, SJ3.1, SJ4.1, U2.REGEN, U2.VCC, U2.VCC@58
- new net N$20: CAM.2, Q4.D
- new net N$21: Q4.G, R20.2, R23.1
- new net N$22: Q3.G, R21.2, R22.1
- new net N$23: Q1.D, R1.2, U$1.EN
- new net N$24: Q1.G, R24.2
- net 3.3V: now also C12.1, C14.1, C15.1, C22.1, C23.+, C25.1, C28.1, D4.C, IC3.AVCC, IC3.VCC, IC3.VCC1, IC3.VCC2, IC3.VCC3, J1.2, Q3.S, Q4.S, R10.2, R16.2, R18.1, R19.2, R2.2, R20.1, R21.1, RN1B.2, RN1C.2, U$1.VOS, U$6.P$2, U4.S1, U4.VDD, U4.VDDIO; no longer C5.1, C6.+, C8.1, CAM.2, L1.1, R3.2, SJ2.1, SJ3.1, SJ4.1, U2.REGEN, U2.VCC, U2.VCC@58
- net GND: now also C28.2, J1.6, JP1.2, Q5.S, Q6.S, R13.2; no longer JP1.1, Q2.S
- net MISO: now also J1.1
- net MOSI: now also J1.4
- net N$10: now also Q6.G; no longer Q1.G
- net N$7: now also Q5.G; no longer Q2.G
- net N$8: now also Q6.D; no longer Q1.D
- net N$9: now also Q5.D; no longer Q2.D
- net RESET: now also J1.5, R19.1; no longer RN5A.1
- net SCK: now also J1.3
- net SCL: no longer U2.SCL
- net SDA: no longer U2.SDA
- net VCC_EN: now also R24.1; no longer R1.2, U$1.EN
- net V_BATT: now also JP1.1; no longer JP1.2, R13.2
Other:
- moved on the sheet: C11, C21, CAM, WIND

Commit message: board version 5.1
Parts:
- removed R10, R2: DNP, SparkFun:RESISTOR0402-RES
- removed R19: 10k, SparkFun-Resistors:RESISTOR0603
- removed U$3: 4.7uH, kolosy:VLCF4020
- removed U$6: 15uH, kolosy:VLCF4020
- added C29: 0.1uF, SparkFun-Passives:CAP0402-CAP
- added C30: (no value), kolosy:CAP_POL
- added JP2: FTDI_DEVICE, SparkFun-Connectors:FTDI_DEVICE
- added L2: 15uH, kolosy:VLCF4020
- added L3: 4.7uH, kolosy:SLF6028
- added R25: 70R, SparkFun-Resistors:RESISTOR0603
- added STATUS: RED, SparkFun-LED:LED-RED0603
- C1, C2, C28, C3, C4: device SparkFun-Passives:CAP0402-CAP -> SparkFun-Passives:CAP0603-CAP
- C17, C20: device SparkFun-Capacitors:CAP0603-CAP -> SparkFun-Capacitors:CAP1206
- C18, C21, C22: device SparkFun-Capacitors:CAP0603-CAP -> SparkFun-Capacitors:CAP0805
- C23: value 200mF -> (none); device SparkFun-Capacitors:CAP_POLEN_J2 -> kolosy:CAP_POL
- C25, C26, C27: device SparkFun:CAP0402-CAP -> SparkFun:CAP0603-CAP
- C9: value DNP -> 250uF; device SparkFun:CAP_POLEN_J2 -> SparkFun-Capacitors:CAPPTH1
Connections:
- removed net PC5: IC3.(A13)PC5
- removed net PE0: IC3.(RXD0/PCIN8)PE0
- removed net PE1: IC3.(TXD0)PE1
- removed net RX0: RN1A.1, U2.RXD0
- new net DTR: C29.1, JP2.DTR
- new net N$25: JP2.CTS
- new net N$27: R25.1, STATUS.C
- new net RX_D0: IC3.(RXD0/PCIN8)PE0, JP2.RXI
- new net STATUS_LED: IC3.(A13)PC5, STATUS.A
- new net TX_D0: IC3.(TXD0)PE1, JP2.TXO
- net 3.3V: now also C9.1, JP2.VCC, L2.P$2, RN1A.2; no longer R10.2, R19.2, R2.2, U$6.P$2
- net 5V: now also L3.P$1; no longer U$3.P$1
- net GND: now also C30.-, C9.2, JP2.GND, R25.2; no longer C9.-
- net N$12: now also L3.P$2; no longer U$3.P$2
- net N$14: now also L2.P$1; no longer U$6.P$1
- net RESET: now also C29.2, RN1A.1; no longer R19.1
- net RXD2: now also U2.TXD0; no longer RN1A.2
- net SCL: no longer R2.1
- net SDA: no longer R10.1
- net TXD2: now also U2.RXD0; no longer U2.TXD0
- net VBAT: now also C30.+; no longer C9.+
Other:
- moved on the sheet: RN1A

Commit message: cleanup
Parts:
- removed SJ1: (no value), SparkFun-Passives:SOLDERJUMPER_2WAYPASTE2&3
- removed SJ2**, SJ3**: SOLDERJUMPERTRACE, SparkFun-Passives:SOLDERJUMPERTRACE
- R25: value 70R -> 100R
Connections:
- removed net AD0: SJ1.2, U1.AD0
- removed net CLKIN: SJ2**.2, U1.CLKIN
- removed net FSYNC: SJ3**.2, U1.FSYNC
- net 3.3V: no longer SJ1.1
- net GND: now also U1.AD0, U1.CLKIN, U1.FSYNC; no longer SJ1.3, SJ2**.1, SJ3**.1
- net INT: now also IC3.PJ3(PCINT12)

Commit message: 5.1 version final; 1A 5V reg
Parts:
- removed SJ4: BAT, SparkFun:SOLDERJUMPERNC
- added Q2, Q8: MOSFET-PCHANNELSMD, SparkFun-DiscreteSemi:MOSFET-PCHANNELSMD
- added Q7: MOSFET-NCHANNELBSS138, SparkFun-DiscreteSemi:MOSFET-NCHANNELBSS138
- added R10, R26: 100R, SparkFun-Resistors:RESISTOR0603
- added R19, R2, R27: 100k, SparkFun-Resistors:RESISTOR0603
- C22: value 10uF -> 22uF
- R11: value 680R -> 100K
- R15: value 31.6k -> 56.2k
- R5: value 2.5K -> 324K
Connections:
- removed net N$6: D1.A, SJ4.2
- removed net PC3: IC3.(A11)PC3
- removed net PC4: IC3.(A12)PC4
- new net BATT_SENS_EN: IC3.(A11)PC3, R26.1
- new net N$26: Q2.D, WIND.2
- new net N$28: Q2.G, R10.1, R2.2
- new net N$29: Q8.D, R5.2
- new net N$30: Q7.D, Q8.G, R19.2
- new net N$31: Q7.G, R26.2, R27.2
- new net WIND_EN: IC3.(A12)PC4, R10.2
- net 3.3V: now also Q2.S, R2.1; no longer WIND.2
- net GND: now also Q7.S, R27.1
- net GPS_PWR: now also D1.A; no longer SJ4.1
- net V_BATT: now also Q8.S, R19.1; no longer R5.2
Other:
- moved on the sheet: C13, C17, C18, C19, C20, C21, C22, C24, C9, CAM, D$1, D$2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

Commit message: 5.1 final; submitted for build
Parts:
- removed D$3: SS1P3L, kolosy:SS1P3L
- removed D5: (no value), diode:DIODE-SOD523
- added C31: 22uF, SparkFun-Capacitors:CAP1206
- added C32: .1uF, SparkFun-Capacitors:CAP0805
- added C33: DNP, SparkFun-Passives:CAP0402-CAP
- C17: value 10uF -> 22uF
- C18: value .01uF -> DNP
- C19: value 1000pF -> .1uF; device SparkFun-Capacitors:CAP0603-CAP -> SparkFun-Capacitors:CAP0805
- L3: device kolosy:SLF6028 -> kolosy:SLF60287055
- R13: value 100k -> 10k
- R14: value 10k -> 56.8K
- R15: value 56.2k -> 10K
- U$2: value LM2374 -> TPS56X200; device kolosy:LM2374 -> kolosy:TPS56X200
Connections:
- removed net N$12: C18.1, D$3.C, L3.P$2, U$2.SW
- new net N$19: C18.2, R14.1, R15.2, U$2.VFB
- new net N$32: C19.2, U$2.VBST
- net 3.3V: now also C33.1
- net 5V: now also C18.1, C31.1, L3.P$2, R14.2; no longer C19.1, D5.A, L3.P$1, R15.2
- net 5V_EN: no longer U$2.EN
- net GND: now also C31.2, C32.2, R15.1; no longer D$3.A, R13.2, R14.1
- net N$11: now also C19.1, L3.P$1, U$2.SW; no longer C18.2, D5.C, U$2.BOOST
- net N$15: now also R13.2, U$2.EN; no longer C19.2, R14.2, R15.1, U$2.FB
- net N$17: now also C33.2
- net V_BATT: now also C32.1
Other:
- note removed: "(see datasheet)"
- note removed: "RX1/TX1 and I2C ports"
- note removed: "SPI port is used for"
- note removed: "are only available via"
- note removed: "custom firmware. Contact"
- note removed: "external Flash memory"
- note removed: "optional logging to"
- note removed: "www.skytraq.com.tw for info."
- moved on the sheet: C17, C18, C19, C20, C22, C9, L3, R13, R14, R15

Commit message: circuit updates, firmware tweaks
Parts:
- added C34: 470uF, SparkFun-Capacitors:CAPPTH1
- C13: value 250uF -> 4700uF
- C24: value 250uF -> 1000uF
Connections:
- net GND: now also C34.2
- net V_BATT: now also C34.1
Changed lines of the file:
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@@
 <?xml version="1.0" encoding="utf-8"?>
 <!DOCTYPE eagle SYSTEM "eagle.dtd">
-<eagle version="6.4">
+<eagle version="7.2.0">
 <drawing>
 <settings>
@@
 <grid distance="0.1" unitdist="inch" unit="inch" style="lines" multiple="1" display="no" altdistance="0.01" altunitdist="inch" altunit="inch"/>
 <layers>
-<layer number="1" name="Top" color="4" fill="1" visible="yes" active="no"/>
-<layer number="16" name="Bottom" color="1" fill="1" visible="yes" active="no"/>
-<layer number="17" name="Pads" color="2" fill="1" visible="yes" active="no"/>
-<layer number="18" name="Vias" color="2" fill="1" visible="yes" active="no"/>
-<layer number="19" name="Unrouted" color="6" fill="1" visible="yes" active="no"/>
-<layer number="20" name="Dimension" color="15" fill="1" visible="yes" active="no"/>
-<layer number="21" name="tPlace" color="7" fill="1" visible="yes" active="no"/>
-<layer number="22" name="bPlace" color="7" fill="1" visible="yes" active="no"/>
-<layer number="23" name="tOrigins" color="15" fill="1" visible="yes" active="no"/>
-<layer number="24" name="bOrigins" color="15" fill="1" visible="yes" active="no"/>
-<layer number="25" name="tNames" color="7" fill="1" visible="yes" active="no"/>
-<layer number="26" name="bNames" color="7" fill="1" visible="yes" active="no"/>
-<layer number="27" name="tValues" color="7" fill="1" visible="yes" active="no"/>
-<layer number="28" name="bValues" color="7" fill="1" visible="yes" active="no"/>
+<layer number="1" name="Top" color="4" fill="1" visible="no" active="no"/>
+<layer number="16" name="Bottom" color="1" fill="1" visible="no" active="no"/>
+<layer number="17" name="Pads" color="2" fill="1" visible="no" active="no"/>
+<layer number="18" name="Vias" color="2" fill="1" visible="no" active="no"/>
+<layer number="19" name="Unrouted" color="6" fill="1" visible="no" active="no"/>
+<layer number="20" name="Dimension" color="15" fill="1" visible="no" active="no"/>
+<layer number="21" name="tPlace" color="7" fill="1" visible="no" active="no"/>
+<layer number="22" name="bPlace" color="7" fill="1" visible="no" active="no"/>
+<layer number="23" name="tOrigins" color="15" fill="1" visible="no" active="no"/>
+<layer number="24" name="bOrigins" color="15" fill="1" visible="no" active="no"/>
+<layer number="25" name="tNames" color="7" fill="1" visible="no" active="no"/>
+<layer number="26" name="bNames" color="7" fill="1" visible="no" active="no"/>
+<layer number="27" name="tValues" color="7" fill="1" visible="no" active="no"/>
+<layer number="28" name="bValues" color="7" fill="1" visible="no" active="no"/>
 <layer number="29" name="tStop" color="7" fill="3" visible="no" active="no"/>
 <layer number="30" name="bStop" color="7" fill="6" visible="no" active="no"/>
@@
 <layer number="35" name="tGlue" color="7" fill="4" visible="no" active="no"/>
 <layer number="36" name="bGlue" color="7" fill="5" visible="no" active="no"/>
-<layer number="37" name="tTest" color="7" fill="1" visible="yes" active="no"/>
-<layer number="38" name="bTest" color="7" fill="1" visible="yes" active="no"/>
+<layer number="37" name="tTest" color="7" fill="1" visible="no" active="no"/>
+<layer number="38" name="bTest" color="7" fill="1" visible="no" active="no"/>
 <layer number="39" name="tKeepout" color="4" fill="11" visible="no" active="no"/>
 <layer number="40" name="bKeepout" color="1" fill="11" visible="no" active="no"/>
@@
 <layer number="44" name="Drills" color="7" fill="1" visible="no" active="no"/>
 <layer number="45" name="Holes" color="7" fill="1" visible="no" active="no"/>
-<layer number="46" name="Milling" color="3" fill="1" visible="yes" active="no"/>
-<layer number="47" name="Measures" color="7" fill="1" visible="yes" active="no"/>
-<layer number="48" name="Document" color="7" fill="1" visible="yes" active="no"/>
-<layer number="49" name="Reference" color="7" fill="1" visible="yes" active="no"/>
-<layer number="50" name="dxf" color="7" fill="1" visible="yes" active="no"/>
-<layer number="51" name="tDocu" color="7" fill="1" visible="yes" active="no"/>
-<layer number="52" name="bDocu" color="7" fill="1" visible="yes" active="no"/>
-<layer number="53" name="tGND_GNDA" color="7" fill="9" visible="yes" active="no"/>
-<layer number="54" name="bGND_GNDA" color="1" fill="9" visible="yes" active="no"/>
-<layer number="56" name="wert" color="7" fill="1" visible="yes" active="no"/>
+<layer number="46" name="Milling" color="3" fill="1" visible="no" active="no"/>
+<layer number="47" name="Measures" color="7" fill="1" visible="no" active="no"/>
+<layer number="48" name="Document" color="7" fill="1" visible="no" active="no"/>
+<layer number="49" name="Reference" color="7" fill="1" visible="no" active="no"/>
+<layer number="50" name="dxf" color="7" fill="1" visible="no" active="no"/>
+<layer number="51" name="tDocu" color="7" fill="1" visible="no" active="no"/>
+<layer number="52" name="bDocu" color="7" fill="1" visible="no" active="no"/>
+<layer number="53" name="tGND_GNDA" color="7" fill="9" visible="no" active="no"/>
+<layer number="54" name="bGND_GNDA" color="1" fill="9" visible="no" active="no"/>
+<layer number="56" name="wert" color="7" fill="1" visible="no" active="no"/>
 <layer number="91" name="Nets" color="2" fill="1" visible="yes" active="yes"/>
 <layer number="92" name="Busses" color="1" fill="1" visible="yes" active="yes"/>
@@
 <part name="GND35" library="supply1" deviceset="GND" device=""/>
 <part name="R1" library="SparkFun-Resistors" deviceset="RESISTOR" device="0603" value="100k"/>
-<part name="C13" library="SparkFun-Capacitors" deviceset="CAP" device="PTH1" value="250uF"/>
-<part name="C24" library="SparkFun-Capacitors" deviceset="CAP" device="PTH1" value="250uF"/>
+<part name="C13" library="SparkFun-Capacitors" deviceset="CAP" device="PTH1" value="4700uF"/>
+<part name="C24" library="SparkFun-Capacitors" deviceset="CAP" device="PTH1" value="1000uF"/>
 <part name="GND17" library="SparkFun-Aesthetics" deviceset="GND" device=""/>
 <part name="GND36" library="SparkFun-Aesthetics" deviceset="GND" device=""/>
@@
 <part name="C18" library="SparkFun-Capacitors" deviceset="CAP" device="0805" value="DNP"/>
 <part name="C33" library="SparkFun-Passives" deviceset="CAP" device="0402-CAP" value="DNP"/>
+<part name="C34" library="SparkFun-Capacitors" deviceset="CAP" device="PTH1" value="470uF"/>
 </parts>
 <sheets>
@@
 <attribute name="VALUE" x="313.436" y="-75.819" size="1.778" layer="96" rot="MR0"/>
 </instance>
+<instance part="C34" gate="G$1" x="203.2" y="-81.28"/>
 </instances>
 <busses>
@@
 <pinref part="U$1" gate="G$1" pin="GND"/>
 <wire x1="241.3" y1="-83.82" x2="226.06" y2="-83.82" width="0.1524" layer="91"/>
+<pinref part="C34" gate="G$1" pin="2"/>
+<wire x1="226.06" y1="-83.82" x2="203.2" y2="-83.82" width="0.1524" layer="91"/>
 </segment>
 <segment>
@@
 <wire x1="226.06" y1="-73.66" x2="226.06" y2="-68.58" width="0.1524" layer="91"/>
 <junction x="226.06" y="-73.66"/>
-</segment>
-</net>
+<pinref part="C34" gate="G$1" pin="1"/>
+<wire x1="203.2" y1="-76.2" x2="203.2" y2="-73.66" width="0.1524" layer="91"/>
+<wire x1="203.2" y1="-73.66" x2="226.06" y2="-73.66" width="0.1524" layer="91"/>
+</segment>
+</net>
