File: layout/boat5.sch (EAGLE design)
At the start: 98 parts, among them IC3 ATMEGA2560-16AU, J1 AVR_SPI_PRG_6PTH, Q1 MOSFET-NCHANNELBSS138, Q2 MOSFET-PCHANNELSMD, Q3 MOSFET-PCHANNELSMD, Q4 MOSFET-PCHANNELSMD, Q5 MOSFET-NCHANNELBSS138, Q6 MOSFET-NCHANNELBSS138, Q7 MOSFET-NCHANNELBSS138, Q8 MOSFET-PCHANNELSMD, U1 MPU-9150, U2 VENUS638FLPX-L, U3 USD-SOCKETNEW, U4 HMC5883LSMD, Y1 CSTCE16M0V53-R0 16MHZ

Commit message: new calibration params, other fixes
Parts:
- C10, C5, C7, C8: device SparkFun:CAP0402-CAP -> SparkFun:CAP0603-CAP
- C18, C33: value DNP -> 1nF
- L1: device SparkFun:INDUCTOR0402 -> SparkFun:INDUCTOR0603
- R3, R4, R6: device SparkFun:RESISTOR0402-RES -> SparkFun:RESISTOR0603-RES
Changed lines of the file:
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@@
 <grid distance="0.1" unitdist="inch" unit="inch" style="lines" multiple="1" display="no" altdistance="0.01" altunitdist="inch" altunit="inch"/>
 <layers>
-<layer number="1" name="Top" color="4" fill="1" visible="no" active="no"/>
-<layer number="16" name="Bottom" color="1" fill="1" visible="no" active="no"/>
-<layer number="17" name="Pads" color="2" fill="1" visible="no" active="no"/>
-<layer number="18" name="Vias" color="2" fill="1" visible="no" active="no"/>
-<layer number="19" name="Unrouted" color="6" fill="1" visible="no" active="no"/>
-<layer number="20" name="Dimension" color="15" fill="1" visible="no" active="no"/>
-<layer number="21" name="tPlace" color="7" fill="1" visible="no" active="no"/>
-<layer number="22" name="bPlace" color="7" fill="1" visible="no" active="no"/>
-<layer number="23" name="tOrigins" color="15" fill="1" visible="no" active="no"/>
-<layer number="24" name="bOrigins" color="15" fill="1" visible="no" active="no"/>
-<layer number="25" name="tNames" color="7" fill="1" visible="no" active="no"/>
-<layer number="26" name="bNames" color="7" fill="1" visible="no" active="no"/>
-<layer number="27" name="tValues" color="7" fill="1" visible="no" active="no"/>
-<layer number="28" name="bValues" color="7" fill="1" visible="no" active="no"/>
+<layer number="1" name="Top" color="4" fill="1" visible="yes" active="no"/>
+<layer number="16" name="Bottom" color="1" fill="1" visible="yes" active="no"/>
+<layer number="17" name="Pads" color="2" fill="1" visible="yes" active="no"/>
+<layer number="18" name="Vias" color="2" fill="1" visible="yes" active="no"/>
+<layer number="19" name="Unrouted" color="6" fill="1" visible="yes" active="no"/>
+<layer number="20" name="Dimension" color="15" fill="1" visible="yes" active="no"/>
+<layer number="21" name="tPlace" color="7" fill="1" visible="yes" active="no"/>
+<layer number="22" name="bPlace" color="7" fill="1" visible="yes" active="no"/>
+<layer number="23" name="tOrigins" color="15" fill="1" visible="yes" active="no"/>
+<layer number="24" name="bOrigins" color="15" fill="1" visible="yes" active="no"/>
+<layer number="25" name="tNames" color="7" fill="1" visible="yes" active="no"/>
+<layer number="26" name="bNames" color="7" fill="1" visible="yes" active="no"/>
+<layer number="27" name="tValues" color="7" fill="1" visible="yes" active="no"/>
+<layer number="28" name="bValues" color="7" fill="1" visible="yes" active="no"/>
 <layer number="29" name="tStop" color="7" fill="3" visible="no" active="no"/>
 <layer number="30" name="bStop" color="7" fill="6" visible="no" active="no"/>
@@
 <layer number="35" name="tGlue" color="7" fill="4" visible="no" active="no"/>
 <layer number="36" name="bGlue" color="7" fill="5" visible="no" active="no"/>
-<layer number="37" name="tTest" color="7" fill="1" visible="no" active="no"/>
-<layer number="38" name="bTest" color="7" fill="1" visible="no" active="no"/>
+<layer number="37" name="tTest" color="7" fill="1" visible="yes" active="no"/>
+<layer number="38" name="bTest" color="7" fill="1" visible="yes" active="no"/>
 <layer number="39" name="tKeepout" color="4" fill="11" visible="no" active="no"/>
 <layer number="40" name="bKeepout" color="1" fill="11" visible="no" active="no"/>
@@
 <layer number="44" name="Drills" color="7" fill="1" visible="no" active="no"/>
 <layer number="45" name="Holes" color="7" fill="1" visible="no" active="no"/>
-<layer number="46" name="Milling" color="3" fill="1" visible="no" active="no"/>
-<layer number="47" name="Measures" color="7" fill="1" visible="no" active="no"/>
-<layer number="48" name="Document" color="7" fill="1" visible="no" active="no"/>
-<layer number="49" name="Reference" color="7" fill="1" visible="no" active="no"/>
-<layer number="50" name="dxf" color="7" fill="1" visible="no" active="no"/>
-<layer number="51" name="tDocu" color="7" fill="1" visible="no" active="no"/>
-<layer number="52" name="bDocu" color="7" fill="1" visible="no" active="no"/>
-<layer number="53" name="tGND_GNDA" color="7" fill="9" visible="no" active="no"/>
-<layer number="54" name="bGND_GNDA" color="1" fill="9" visible="no" active="no"/>
-<layer number="56" name="wert" color="7" fill="1" visible="no" active="no"/>
+<layer number="46" name="Milling" color="3" fill="1" visible="yes" active="no"/>
+<layer number="47" name="Measures" color="7" fill="1" visible="yes" active="no"/>
+<layer number="48" name="Document" color="7" fill="1" visible="yes" active="no"/>
+<layer number="49" name="Reference" color="7" fill="1" visible="yes" active="no"/>
+<layer number="50" name="dxf" color="7" fill="1" visible="yes" active="no"/>
+<layer number="51" name="tDocu" color="7" fill="1" visible="yes" active="no"/>
+<layer number="52" name="bDocu" color="7" fill="1" visible="yes" active="no"/>
+<layer number="53" name="tGND_GNDA" color="7" fill="9" visible="yes" active="no"/>
+<layer number="54" name="bGND_GNDA" color="1" fill="9" visible="yes" active="no"/>
+<layer number="56" name="wert" color="7" fill="1" visible="yes" active="no"/>
 <layer number="91" name="Nets" color="2" fill="1" visible="yes" active="yes"/>
 <layer number="92" name="Busses" color="1" fill="1" visible="yes" active="yes"/>
@@
 <part name="GND23" library="SparkFun" deviceset="GND" device=""/>
 <part name="GND6" library="SparkFun" deviceset="GND" device=""/>
-<part name="R3" library="SparkFun" deviceset="RESISTOR" device="0402-RES" value="33k"/>
-<part name="C5" library="SparkFun" deviceset="CAP" device="0402-CAP" value="0.1uF"/>
+<part name="R3" library="SparkFun" deviceset="RESISTOR" device="0603-RES" value="33k"/>
+<part name="C5" library="SparkFun" deviceset="CAP" device="0603-CAP" value="0.1uF"/>
 <part name="C6" library="SparkFun" deviceset="CAP_POL" device="1206" value="10uF"/>
-<part name="R4" library="SparkFun" deviceset="RESISTOR" device="0402-RES" value="10k"/>
+<part name="R4" library="SparkFun" deviceset="RESISTOR" device="0603-RES" value="10k"/>
 <part name="GND10" library="SparkFun" deviceset="GND" device=""/>
 <part name="GND11" library="SparkFun" deviceset="GND" device=""/>
-<part name="C7" library="SparkFun" deviceset="CAP" device="0402-CAP" value="1uF"/>
+<part name="C7" library="SparkFun" deviceset="CAP" device="0603-CAP" value="1uF"/>
 <part name="GND12" library="SparkFun" deviceset="GND" device=""/>
 <part name="SJ2" library="SparkFun" deviceset="SOLDERJUMPER_2WAY" device="PASTE2&amp;3" value="BTS"/>
 <part name="GND13" library="SparkFun" deviceset="GND" device=""/>
 <part name="SJ3" library="SparkFun" deviceset="SOLDERJUMPER_2WAY" device="PASTE2&amp;3" value="PSE"/>
-<part name="L1" library="SparkFun" deviceset="INDUCTOR" device="0402" value="33nH"/>
-<part name="C8" library="SparkFun" deviceset="CAP" device="0402-CAP" value="22pF"/>
+<part name="L1" library="SparkFun" deviceset="INDUCTOR" device="0603" value="33nH"/>
+<part name="C8" library="SparkFun" deviceset="CAP" device="0603-CAP" value="22pF"/>
 <part name="JP5" library="SparkFun" deviceset="SMA_EDGE" device=""/>
 <part name="U2" library="mike-temp" deviceset="VENUS638FLPX-L" device=""/>
@@
 <part name="GND14" library="SparkFun" deviceset="GND" device=""/>
 <part name="D1" library="SparkFun" deviceset="DIODE" device="SOD" value="BAS16"/>
-<part name="R6" library="SparkFun" deviceset="RESISTOR" device="0402-RES" value="330"/>
+<part name="R6" library="SparkFun" deviceset="RESISTOR" device="0603-RES" value="330"/>
 <part name="GND15" library="SparkFun" deviceset="GND" device=""/>
-<part name="C10" library="SparkFun" deviceset="CAP" device="0402-CAP" value="0.1uF"/>
+<part name="C10" library="SparkFun" deviceset="CAP" device="0603-CAP" value="0.1uF"/>
 <part name="GND16" library="SparkFun" deviceset="GND" device=""/>
 <part name="JP1" library="SparkFun-Connectors" deviceset="M03" device="SCREW"/>
@@
 <part name="C31" library="SparkFun-Capacitors" deviceset="CAP" device="1206" value="22uF"/>
 <part name="C32" library="SparkFun-Capacitors" deviceset="CAP" device="0805" value=".1uF"/>
-<part name="C18" library="SparkFun-Capacitors" deviceset="CAP" device="0805" value="DNP"/>
-<part name="C33" library="SparkFun-Passives" deviceset="CAP" device="0402-CAP" value="DNP"/>
+<part name="C18" library="SparkFun-Capacitors" deviceset="CAP" device="0805" value="1nF"/>
+<part name="C33" library="SparkFun-Passives" deviceset="CAP" device="0402-CAP" value="1nF"/>
 <part name="C34" library="SparkFun-Capacitors" deviceset="CAP" device="PTH1" value="470uF"/>
 </parts>
