File: layout/boat7.sch (EAGLE design)
At the start: 118 parts, among them IC3 ATMEGA2560-16AU, J1 AVR_SPI_PRG_6PTH, J2 POWER_JACKPTH, J3 POWER_JACKPTH, Q1 200mA/50V, Q2 MOSFET-PCHANNELSMD, Q3 MOSFET-PCHANNELSMD, Q4 MOSFET-PCHANNELSMD, Q5 200mA/50V, Q6 200mA/50V, Q7 200mA/50V, Q8 MOSFET-PCHANNELSMD, Q9 MOSFET-PCHANNELSMD, U1 MPU-9150, U2 VENUS638FLPX-L, U3 USD-SOCKETNEW, Y1 CSTCE16M0V53-R0 16MHZ

Commit message: Finalized v7 board layout / schematic
Parts:
- removed C24: 1000uF, SparkFun-Capacitors:CAPPTH1
- removed C3: 10nF, SparkFun-Passives:CAP0603-CAP
- removed C4: 0.1uF, SparkFun-Passives:CAP0603-CAP
- removed D8: MBRS340, kolosy:MBRS340
- added D3: MBRA340T3, diode:MBRA340T3
- added R38: FUSE, SparkFun-Resistors:RESISTORPTH-1/4W-VERT
- added R40: 10K, SparkFun-Resistors:10KOHM-1/10W-1%(0603)0603
- C1: device SparkFun-Passives:CAP0603-CAP -> SparkFun-Capacitors:0.1UF-25V(+80/-20%)(0603)
- C2: value 2.2nF -> 0.1uF; device SparkFun-Passives:CAP0603-CAP -> SparkFun-Capacitors:0.1UF-25V(+80/-20%)(0603)
- C29: device SparkFun-Passives:CAP0402-CAP -> SparkFun-Passives:CAP0603-CAP
- C9: value 250uF -> 470uF
- U1: value MPU-9150 -> MPU-9250; device SparkFun-Sensors:MPU-9150QFN-24-NP -> Testing:MPU-9250
Connections:
- removed net CLKOUT: U1.CLKOUT
- removed net ESC: U1.E_SCL
- removed net ESD: U1.E_SDA
- removed net N$2: C4.1, U1.REGOUT
- new net !CS: R40.1, RN1D.1, U1.!CS
- new net AUX_CL: U1.AUX_CL
- new net AUX_DA: U1.AUX_DA
- new net FSYNC: U1.FSYNC
- new net REGOUT: C1.1, U1.REGOUT
- net 3.3V: now also C2.1, R40.2, RN1D.2, U1.VDD, U1.VDDIO; no longer C1.1, C3.1, U1.VDD@13, U1.VDD@3, U1.VLOGIC
- net 5V: now also R38.2; no longer C24.1, S_WINCH.2
- net GND: now also D3.A, U1.AD0/SDO, U1.GND; no longer C24.2, C3.2, C4.2, D8.A, U1.AD0, U1.CLKIN, U1.FSYNC, U1.GND@15, U1.GND@17, U1.GND@18
- net N$1: now also R38.1, S_WINCH.2; no longer C2.1, U1.CPOUT
- net SCL: now also U1.SCL/SCLK; no longer U1.SCL
- net SDA: now also U1.SDA/SDI; no longer U1.SDA
- net SW: now also D3.C; no longer D8.K
Other:
- note added: "AD0 sets LSB of address"
- note added: "AD0/SDO defaults to 0V. This sets the I2C address to 0b1101000 (0x68) and leaves the AD0/SDO PTH disconnected. Connect to AD0/SD0 PTH to change externally. Pull high to set address to 0b1101001 (0x69)."
- note removed: "50V"
- note removed: "I2C Address Selection"
- note removed: "default to GND"
- moved on the sheet: C1, C13, C2, RN1D
