File: layout/boat7.brd (EAGLE design)
At the start: 101.6 x 53.3 mm, 118 parts, among them IC3 ATMEGA2560-16AU, J1 AVR_SPI_PRG_6PTH, J2 POWER_JACKPTH, J3 POWER_JACKPTH, Q1 200mA/50V, Q2 MOSFET-PCHANNELSMD, Q3 MOSFET-PCHANNELSMD, Q4 MOSFET-PCHANNELSMD, Q5 200mA/50V, Q6 200mA/50V, Q7 200mA/50V, Q8 MOSFET-PCHANNELSMD, Q9 MOSFET-PCHANNELSMD, U1 MPU-9150, U2 VENUS638FLPX-L, U3 USD-SOCKETNEW, Y1 CSTCE16M0V53-R0 16MHZ

Commit message: Finalized v7 board layout / schematic
Parts:
- removed C24: 1000uF, SparkFun-Capacitors:CAP-PTH-5MM
- removed C3: 10nF, SparkFun-Passives:0603-CAP
- removed C4: 0.1uF, SparkFun-Passives:0603-CAP
- removed D8: MBRS340, kolosy:DO214BA
- added D3: MBRA340T3, diode:SMA
- added R38: FUSE, SparkFun-Resistors:AXIAL-0.1
- added R40: 10K, SparkFun-Resistors:0603-RES
- C1: device SparkFun-Passives:0603-CAP -> SparkFun-Capacitors:0603-CAP
- C2: value 2.2nF -> 0.1uF; device SparkFun-Passives:0603-CAP -> SparkFun-Capacitors:0603-CAP
- C29: device SparkFun-Passives:0402-CAP -> SparkFun-Passives:0603-CAP
- C9: value 250uF -> 470uF
- U1: value MPU-9150 -> MPU-9250; device SparkFun-Sensors:QFN-24-NP -> Testing:QFN24_PAD
- moved C13 12.0 mm to (59.0, 40.6), turned to 0 degrees
- moved C1 5.89 mm to (57.1, 2.50), turned to 270 degrees
- moved C2 4.65 mm to (59.1, 5.75)
- moved D$1 2.69 mm to (53.2, 46.4), turned to 90 degrees
- moved R8 1.00 mm to (70.4, 47.6)
- moved C20 0.75 mm to (81.7, 48.7)
- moved C31 0.75 mm to (81.7, 46.6)
- moved R26 0.70 mm to (40.2, 6.95)
- moved R100 0.60 mm to (36.8, 6.95), turned to 180 degrees
- moved CAM 0.45 mm to (63.0, 21.9)
- moved Y1 0.40 mm to (41.7, 12.8)
- moved R17 0.35 mm to (25.1, 3.00)
- moved U1 0.29 mm to (56.5, 5.95)
- moved C23 0.29 mm to (87.4, 5.20)
- moved U$15 0.20 mm to (91.2, 5.00)
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Connections:
- net ESC renamed AUX_CL
- removed net CLKOUT: U1.22
- removed net ESD: U1.6
- removed net N$2: C4.1, U1.10
- new net !CS: R40.1, RN1.4, U1.22
- new net AUX_DA: U1.21
- new net FSYNC: U1.11
- new net REGOUT: C1.1, U1.10
- net 3.3V: now also C2.1, R40.2, RN1.5, U1.1; no longer C1.1, C3.1, U1.3
- net 5V: now also R38.P$2; no longer C24.1, S_WINCH.2
- net GND: now also D3.A, U1.20, U1.CENTER; no longer C24.2, C3.2, C4.2, D8.A, U1.1, U1.11, U1.15, U1.17
- net N$1: now also R38.P$1, S_WINCH.2; no longer C2.1, U1.20
- net SW: now also D3.C; no longer D8.C
Routing:
- net !CS: track 0.00 -> 24.5 mm, vias 0 -> 4
- net GND: track 44.7 -> 58.9 mm, vias 50 -> 53
- net RXD3: track 46.6 -> 41.5 mm, vias 3 -> 1
- net 3.3V: track 262.7 -> 266.9 mm, vias 12 -> 13
- net N$1: track 1.55 -> 4.56 mm
- net INT: track 38.4 -> 35.6 mm, vias 3 -> 2
- net GPS_PWR: track 51.4 -> 54.0 mm
- net MOSI: track 30.3 -> 27.9 mm
- net 5V_EN: track 52.6 -> 50.3 mm, vias 4 -> 2
- net VCC_EN: track 46.3 -> 48.3 mm
- net N$2: track 1.96 -> 0.00 mm
- net WINCH_EN: track 24.3 -> 22.4 mm
- net V_BATT_DIV: track 42.4 -> 44.1 mm
- net CS: track 54.7 -> 53.0 mm
- net RXD1: track 33.7 -> 32.1 mm
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
Commit message: new route + additional components
Routing:
- net GND: vias 53 -> 54
Changed lines of the file:
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@@
 <wire x1="59.975" y1="7.175" x2="59.975" y2="6.975" width="0.254" layer="1"/>
 <contactref element="D3" pad="A"/>
+<via x="15" y="21" extent="1-16" drill="0.381"/>
 </signal>
 <signal name="SDA">
@@
 <polygon width="0.254" layer="1" thermals="no">
 <vertex x="24.25" y="14.75"/>
-<vertex x="28.75" y="14.75"/>
-<vertex x="31.1" y="12.4"/>
+<vertex x="27.75" y="14.75"/>
+<vertex x="31.1" y="11.4"/>
 <vertex x="31.1" y="9.35"/>
 <vertex x="24.1" y="9.35"/>
@@
 <wire x1="33" y1="13.75" x2="33" y2="14" width="1.016" layer="16"/>
 <wire x1="33" y1="14" x2="33" y2="15" width="1.016" layer="16"/>
-<wire x1="33" y1="15" x2="40" y2="22" width="1.016" layer="16"/>
+<wire x1="33" y1="15" x2="39.4" y2="21.4" width="1.016" layer="16"/>
 <via x="43" y="25" extent="1-16" drill="0.6"/>
-<wire x1="40" y1="22" x2="43" y2="25" width="1.016" layer="16"/>
+<wire x1="39.4" y1="21.4" x2="43" y2="25" width="1.016" layer="16"/>
 <wire x1="43" y1="25" x2="43" y2="27.3" width="0.3048" layer="1"/>
 <wire x1="38.85" y1="26.15" x2="34.9" y2="26.15" width="0.3048" layer="1"/>
@@
 <wire x1="25" y1="14" x2="25" y2="13.530765625" width="0.4064" layer="1"/>
 <wire x1="25" y1="13.530765625" x2="23.461628125" y2="11.99239375" width="0.4064" layer="1"/>
-<wire x1="25" y1="14" x2="14.48" y2="24.52" width="0.4064" layer="1"/>
-<wire x1="14.48" y1="24.52" x2="12.13" y2="24.52" width="0.4064" layer="1"/>
 <contactref element="U1" pad="13"/>
 <contactref element="C2" pad="1"/>
@@
 <wire x1="54.15" y1="3.85" x2="55" y2="3" width="0.4064" layer="1"/>
 <wire x1="58.65" y1="26.55" x2="58.85" y2="26.75" width="0.6096" layer="1"/>
-<wire x1="39.4" y1="16.65" x2="39.4" y2="19.4" width="0.254" layer="1"/>
-<wire x1="39.4" y1="19.4" x2="40" y2="20" width="0.254" layer="1"/>
-<wire x1="40" y1="20" x2="40" y2="22" width="0.254" layer="1"/>
-<via x="40" y="22" extent="1-16" drill="0.6"/>
 <wire x1="33.289" y1="26.15" x2="34.9" y2="26.15" width="0.3048" layer="1"/>
-<wire x1="38.85" y1="26.15" x2="40" y2="25" width="0.3048" layer="1"/>
-<wire x1="40" y1="25" x2="40" y2="22" width="0.3048" layer="1"/>
+<wire x1="24" y1="14" x2="25" y2="14" width="0.4064" layer="1"/>
+<wire x1="39.4" y1="16.65" x2="39.4" y2="21.4" width="0.254" layer="1"/>
+<wire x1="39.4" y1="21.4" x2="39.4" y2="25.6" width="0.254" layer="1"/>
+<wire x1="39.4" y1="25.6" x2="38.85" y2="26.15" width="0.254" layer="1"/>
+<via x="39.4" y="21.4" extent="1-16" drill="0.381"/>
+<wire x1="24" y1="14" x2="13.48" y2="24.52" width="0.4064" layer="1"/>
+<wire x1="13.48" y1="24.52" x2="12.13" y2="24.52" width="0.4064" layer="1"/>
 </signal>
 <signal name="MOSI">
@@
 <wire x1="29.41" y1="20.11" x2="29.44" y2="20.11" width="0.254" layer="1"/>
 <via x="24.15" y="18.85" extent="1-16" drill="0.381"/>
-<wire x1="24.15" y1="18.85" x2="15.15" y2="18.85" width="0.254" layer="16"/>
-<wire x1="15.15" y1="18.85" x2="11" y2="23" width="0.254" layer="16"/>
+<wire x1="24.15" y1="18.85" x2="15.15" y2="18.85" width="0.3048" layer="16"/>
+<wire x1="15.15" y1="18.85" x2="11" y2="23" width="0.3048" layer="16"/>
 <via x="11" y="23" extent="1-16" drill="0.381"/>
-<wire x1="11" y1="23" x2="11.42" y2="23.42" width="0.254" layer="1"/>
-<wire x1="11.42" y1="23.42" x2="12.33" y2="23.42" width="0.254" layer="1"/>
+<wire x1="11" y1="23" x2="11.42" y2="23.42" width="0.3048" layer="1"/>
+<wire x1="11.42" y1="23.42" x2="12.33" y2="23.42" width="0.3048" layer="1"/>
 </signal>
 <signal name="MISO">
@@
 <contactref element="C21" pad="1"/>
 <contactref element="R1" pad="1"/>
-<wire x1="17.1" y1="5.35" x2="20.8" y2="5.35" width="1.016" layer="1"/>
+<wire x1="17.1" y1="5.35" x2="20.8" y2="5.35" width="1.4224" layer="1"/>
 <wire x1="20.25" y1="3.35" x2="19.1" y2="3.35" width="0.254" layer="1"/>
 <polygon width="0.254" layer="1" thermals="no">
@@
 </polygon>
 <wire x1="19.1" y1="3.35" x2="17.1" y2="5.35" width="0.254" layer="1"/>
-<wire x1="17.1" y1="5.35" x2="13.25" y2="5.35" width="1.016" layer="1"/>
-<wire x1="13.25" y1="5.35" x2="10.75" y2="7.85" width="1.016" layer="1"/>
+<wire x1="17.1" y1="5.35" x2="13.25" y2="5.35" width="1.4224" layer="1"/>
+<wire x1="13.25" y1="5.35" x2="10.75" y2="7.85" width="1.4224" layer="1"/>
 <via x="95" y="36" extent="1-16" drill="0.6" shape="square"/>
 <via x="95" y="34" extent="1-16" drill="0.6" shape="square"/>
@@
 <via x="63" y="8" extent="1-16" drill="0.381"/>
 <via x="63" y="9" extent="1-16" drill="0.381"/>
-<wire x1="81" y1="12.85" x2="81" y2="16.15" width="0.4064" layer="1"/>
+<wire x1="81" y1="12.85" x2="81" y2="16.15" width="0.8128" layer="1"/>
 <wire x1="81" y1="16.15" x2="80.85" y2="16.15" width="0.4064" layer="1"/>
-<wire x1="80.85" y1="16.15" x2="80" y2="17" width="0.4064" layer="1"/>
-<wire x1="80" y1="17" x2="75.1" y2="17" width="0.4064" layer="1"/>
-<wire x1="75.1" y1="17" x2="73.9" y2="18.2" width="0.4064" layer="1"/>
+<wire x1="80.85" y1="16.15" x2="80" y2="17" width="0.8128" layer="1"/>
+<wire x1="80" y1="17" x2="75.1" y2="17" width="0.8128" layer="1"/>
+<wire x1="75.1" y1="17" x2="73.9" y2="18.2" width="0.8128" layer="1"/>
 <via x="97" y="36" extent="1-16" drill="0.6" shape="square"/>
 <via x="97" y="34" extent="1-16" drill="0.6" shape="square"/>
